Commit message: update

File: src/Quadruped-Control-OCS2-ROS2/legged_control/mujoco_simulator/models/quad_mini/urdf/robot.urdf (robot description, URDF)
Before this commit: robot a1, 21 links, 20 joints
Joints:
- joint LF_HFE: axis 0 -1 0 -> 0 1 0
- joint LF_KFE: axis 0 -1 0 -> 0 1 0; limit lower=-0.043633 upper=1.745529 effort=12 velocity=17.80 -> lower=-1.745529 upper=1.745529 effort=12 velocity=17.80
- joint LH_HAA: axis -1 0 0 -> 1 0 0
- joint LH_HFE: axis 0 -1 0 -> 0 1 0
- joint LH_KFE: axis 0 -1 0 -> 0 1 0; limit lower=-0.043633 upper=1.745529 effort=12 velocity=17.80 -> lower=-1.745529 upper=1.745529 effort=12 velocity=17.80
- joint RF_KFE: axis 0 -1 0 -> 0 1 0; limit lower=-0.043633 upper=1.745529 effort=12 velocity=17.80 -> lower=-1.745529 upper=1.745529 effort=12 velocity=17.80
- joint RH_HAA: axis -1 0 0 -> 1 0 0
- joint RH_KFE: axis 0 -1 0 -> 0 1 0; limit lower=-0.043633 upper=1.745529 effort=12 velocity=17.80 -> lower=-1.745529 upper=1.745529 effort=12 velocity=17.80

Commit message: changed urdf axises

File: src/Quadruped-Control-OCS2-ROS2/legged_control/mujoco_simulator/models/quad_mini/urdf/robot.urdf (robot description, URDF)
Before this commit: robot quad_mini, 21 links, 20 joints
Joints:
- joint LF_HFE: axis 0 1 0 -> 0 -1 0
- joint LF_KFE: axis 0 1 0 -> 0 -1 0
- joint LH_HAA: axis 1 0 0 -> -1 0 0
- joint LH_HFE: axis 0 1 0 -> 0 -1 0
- joint LH_KFE: axis 0 1 0 -> 0 -1 0
- joint RF_KFE: axis 0 1 0 -> 0 -1 0
- joint RH_HAA: axis 1 0 0 -> -1 0 0
- joint RH_KFE: axis 0 1 0 -> 0 -1 0
