Commit message: new control mode and msg

File: src/Quadruped-Control-OCS2-ROS2/legged_control/mujoco_simulator/models/quad_mini_real/urdf/robot.urdf (robot description, URDF)
Before this commit: robot quad_mini, 19 links, 18 joints
Joints:
- joint RF_KFE: axis 0 -1 0 -> 0 1 0
- joint RH_KFE: axis 0 -1 0 -> 0 1 0
