Commit message: test

File: src/one_leg_pinocchio_control/urdf/bacak_test_description.urdf (robot description, URDF)
Before this commit: robot bacak_test_description, 13 links, 12 joints
Links:
- link fl_hipx: mass 0.053338 -> 0.803338
- link fl_hipy: mass 0.15008 -> 0.9008
- link fl_knee: mass 0.030068 -> 0.0800068
Joints:
- joint fl_hipx_joint: axis 0 -1 0 -> 0 1 0
